Commit message: added modified liosam for microstrain

File: launch/include/config/robot.urdf.xacro (robot description, xacro)
@@ -21,4 +21,10 @@
     <origin xyz="0 0 0" rpy="0 0 0" />
   </joint>
+  <link name="hesai_lidar"> </link>
+  <joint name="hesai_lidar_joint" type="fixed">
+    <parent link="chassis_link" />
+    <child link="hesai_lidar" />
+    <origin xyz="0 0 0" rpy="0 0 0" />
+  </joint>
   <link name="navsat_link"> </link>
   <joint name="navsat_joint" type="fixed">
